File: VolcaModularMidi.sch (KiCad schematic (older format))
At the start: 6 parts, among them J1 Conn_01x04_Male, J2 DIN-5_180degree, U1 6N139

Commit message: Version 0.1 finished
Parts:
- J2: value DIN-5_180degree -> MIDI_IN
Changed lines of the file:
@@
 P 1500 2600
 F 0 "J2" H 1500 2326 50  0000 C CNN
-F 1 "DIN-5_180degree" H 1500 2235 50  0000 C CNN
+F 1 "MIDI_IN" H 1500 2235 50  0000 C CNN
 F 2 "SensaiLib:din-5" H 1500 2600 50  0001 C CNN
 F 3 "http://www.mouser.com/ds/2/18/40_c091_abd_e-75918.pdf" H 1500 2600 50  0001 C CNN
